File: KiCad/Air Flow Sensor Module.sch (KiCad schematic (older format))
At the start: 18 parts, among them Q1 TIP122, U1 LM358, U2 4N32

Commit message: Replaced component R2 footprint to allow for resistor size of proper wattage
Parts:
- R2: footprint Resistors_THT:R_Axial_DIN0411_L9.9mm_D3.6mm_P20.32mm_Horizontal -> Resistors_THT:R_Axial_DIN0414_L11.9mm_D4.5mm_P20.32mm_Horizontal
Changed lines of the file:
@@
 F 0 "R2" V 5980 4650 50  0000 C CNN
 F 1 "68R" V 5900 4650 50  0000 C CNN
-F 2 "Resistors_THT:R_Axial_DIN0411_L9.9mm_D3.6mm_P20.32mm_Horizontal" V 5830 4650 50  0001 C CNN
+F 2 "Resistors_THT:R_Axial_DIN0414_L11.9mm_D4.5mm_P20.32mm_Horizontal" V 5830 4650 50  0001 C CNN
 F 3 "" H 5900 4650 50  0000 C CNN
 	1    5900 4650
